File: corne-light/pcb/corne-light.kicad_pcb (KiCad board)
At the start: 2 copper layers, 275.5 x 105.6 mm, 122 parts, among them J1 MJ-4PP-9, J2 OLED, J5 Breakaway_Tabs, J6 MJ-4PP-9, J7 OLED, SW1 SW_PUSH, SW10 SW_PUSH, SW11 SW_PUSH, SW12 SW_PUSH, SW13 SW_PUSH, SW14 SW_PUSH, SW15 SW_PUSH, SW16 SW_PUSH, SW17 SW_PUSH, SW18 SW_PUSH, SW19 SW_PUSH, SW2 SW_PUSH, SW20 SW_PUSH, SW21 SW_PUSH, SW22 SW_PUSH, SW23 SW_PUSH, SW24 SW_PUSH, SW25 SW_PUSH, SW26 SW_PUSH, SW27 SW_PUSH, SW28 SW_PUSH, SW29 SW_PUSH, SW3 SW_PUSH, SW30 SW_PUSH, SW31 SW_PUSH, SW32 SW_PUSH, SW33 SW_PUSH, SW34 SW_PUSH, SW35 SW_PUSH, SW36 SW_PUSH, SW37 SW_PUSH, SW38 SW_PUSH, SW39 SW_PUSH, SW4 SW_PUSH, SW40 SW_PUSH, SW41 SW_PUSH, SW42 SW_PUSH, SW5 SW_PUSH, SW6 SW_PUSH, SW7 SW_PUSH, SW8 SW_PUSH, SW9 SW_PUSH, U1 ProMicro, U2 ProMicro

Commit message: [REL] KA v1
Parts:
- removed the G*** at (60.2, 90.9)
- removed the G*** at (60.0, 90.9)
- removed the J5 at (22.2, 93.4)
- removed the J5 at (60.2, 93.4)
- removed the Ref** at (193.2, 51.9)
- removed the Ref** at (179.5, 99.4)
- removed the Ref** at (226.1, 91.7)
- removed the Ref** at (269.2, 55.4)
- removed the Ref** at (269.2, 74.4)
- removed the Ref** at (50.7, 74.4)
- removed the Ref** at (50.7, 55.4)
- removed the Ref** at (250.2, 74.4)
- removed the Ref** at (250.2, 55.4)
- removed the Ref** at (31.7, 74.4)
- removed the Ref** at (107.7, 51.9)
- removed the Ref** at (31.7, 55.4)
- removed the Ref** at (74.8, 91.7)
- removed the Ref** at (121.4, 99.3)
- added ?: , , F.Cu at (107.7, 51.9)
- added ?: , , F.Cu at (50.7, 93.4)
- added ?: , , F.Cu at (269.2, 55.4)
- added ?: , , F.Cu at (121.4, 118.3)
- added ?: , , F.Cu at (179.5, 99.4)
- added ?: , , F.Cu at (31.7, 93.4)
- added ?: , , F.Cu at (250.2, 74.4)
- added ?: , , F.Cu at (31.7, 74.4)
- added ?: , , F.Cu at (50.7, 74.4)
- added ?: , , F.Cu at (226.1, 91.7)
- added ?: , , F.Cu at (50.7, 55.4)
- added ?: , , F.Cu at (31.7, 55.4)
- added ?: , , F.Cu at (250.2, 55.4)
- added ?: , , F.Cu at (269.2, 74.4)
- added ?: , , F.Cu at (193.2, 51.9)
- added D13: D, kbd:D3_TH_SMD_v2, B.Cu at (30.2, 102.9)
- added D14: D, kbd:D3_TH_SMD_v2, B.Cu at (33.2, 102.9)
- added D15: D, kbd:D3_TH_SMD_v2, B.Cu at (68.2, 97.9)
- added D16: D, kbd:D3_TH_SMD_v2, B.Cu at (71.2, 97.9)
- added D17: D, kbd:D3_TH_SMD_v2, B.Cu at (106.2, 97.9)
- added D18: D, kbd:D3_TH_SMD_v2, B.Cu at (109.2, 97.9)
- added G***: LOGO, kbd:corne-logo-horizontal, F.Cu at (65.7, 109.9)
- added G***: LOGO, kdkb_tools:logo-vsmall, F.Cu at (232.7, 90.7)
- added G***: LOGO, kdkb_tools:logo-vsmall, F.Cu at (56.7, 109.7)
- added G***: LOGO, kdkb_tools:logo-vsmall, B.Cu at (232.7, 90.7)
- added G***: LOGO, kbd:corne-logo-horizontal, B.Cu at (65.5, 109.9)
- added G***: LOGO, kdkb_tools:logo-vsmall, B.Cu at (56.7, 109.7)
- added J5: Breakaway_Tabs, kbd:Breakaway_Tabs, F.Cu at (60.2, 112.4)
- added J5: Breakaway_Tabs, kbd:Breakaway_Tabs, F.Cu at (22.2, 112.4)
- added Ref**: Val**, kbd:thread_m2, B.Cu at (31.7, 55.4)
- added Ref**: Val**, kbd:thread_m2, B.Cu at (31.7, 74.4)
- added Ref**: Val**, kbd:thread_m2, B.Cu at (121.4, 118.3)
- added Ref**: Val**, kbd:thread_m2, B.Cu at (226.1, 91.7)
- added Ref**: Val**, kbd:thread_m2, B.Cu at (269.2, 74.4)
- added Ref**: Val**, kbd:thread_m2, B.Cu at (193.2, 51.9)
- added Ref**: Val**, kbd:thread_m2, B.Cu at (269.2, 55.4)
- added Ref**: Val**, kbd:thread_m2, B.Cu at (50.7, 55.4)
- added Ref**: Val**, kbd:thread_m2, B.Cu at (50.7, 93.4)
- added Ref**: Val**, kbd:thread_m2, B.Cu at (250.2, 55.4)
- added Ref**: Val**, kbd:thread_m2, B.Cu at (250.2, 74.4)
- added Ref**: Val**, kbd:thread_m2, B.Cu at (179.5, 99.4)
- added Ref**: Val**, kbd:thread_m2, B.Cu at (107.7, 51.9)
- added Ref**: Val**, kbd:thread_m2, B.Cu at (50.7, 74.4)
- added Ref**: Val**, kbd:thread_m2, B.Cu at (31.7, 93.4)
- added SW13: SW_PUSH, kbd:keyswitch_cherrymx_alps_choc12_1u, F.Cu at (22.2, 102.9)
- added SW14: SW_PUSH, kbd:keyswitch_cherrymx_alps_choc12_1u, F.Cu at (41.2, 102.9)
- added SW15: SW_PUSH, kbd:keyswitch_cherrymx_alps_choc12_1u, F.Cu at (60.2, 98.2)
- added SW16: SW_PUSH, kbd:keyswitch_cherrymx_alps_choc12_1u, F.Cu at (79.2, 95.8)
- added SW17: SW_PUSH, kbd:keyswitch_cherrymx_alps_choc12_1u, F.Cu at (98.2, 98.2)
- added SW18: SW_PUSH, kbd:keyswitch_cherrymx_alps_choc12_1u, F.Cu at (117.2, 100.7)
- moved D19 19.0 mm to (80.5, 117.9)
- moved D20 19.0 mm to (96.7, 117.9)
- moved D21 19.0 mm to (99.7, 117.9)
- moved SW19 19.0 mm to (88.7, 117.8)
- moved SW20 19.0 mm to (109.7, 120.5)
- moved SW21 19.0 mm to (131.9, 124.3)
- moved G*** 0.94 mm to (241.9, 91.0)
- moved G*** 0.94 mm to (241.7, 91.0)
Routing:
- net row2: track 153.9 -> 270.5 mm
- net Net-(D16-Pad2): track 35.7 -> 70.4 mm
- net col0: track 182.3 -> 211.6 mm
- net Net-(D14-Pad2): track 27.9 -> 55.7 mm
- net Net-(D18-Pad2): track 26.7 -> 52.2 mm
- net row3: track 94.6 -> 119.0 mm
- net col3: track 141.3 -> 164.2 mm
- net col4: track 119.9 -> 142.7 mm
- net col2: track 135.2 -> 157.6 mm
- net col1: track 156.5 -> 178.2 mm
- net col5: track 104.9 -> 126.2 mm
- net Net-(D15-Pad2): track 21.3 -> 42.6 mm
- net Net-(D13-Pad2): track 21.1 -> 42.2 mm
- net Net-(D17-Pad2): track 21.1 -> 29.0 mm
- net Net-(D19-Pad2): track 28.1 -> 28.8 mm
Other:
- board size 275.5 x 105.6 mm -> 329.2 x 124.6 mm
- board text removed: "Corne Light v2.0 PCB Designed by foostan"
