File: corne-light/pcb/corne-light.kicad_pcb (KiCad board)
At the start: 2 copper layers, 275.5 x 105.6 mm, 122 parts, among them J1 MJ-4PP-9, J2 OLED, J5 Breakaway_Tabs, J6 MJ-4PP-9, J7 OLED, SW1 SW_PUSH, SW10 SW_PUSH, SW11 SW_PUSH, SW12 SW_PUSH, SW13 SW_PUSH, SW14 SW_PUSH, SW15 SW_PUSH, SW16 SW_PUSH, SW17 SW_PUSH, SW18 SW_PUSH, SW19 SW_PUSH, SW2 SW_PUSH, SW20 SW_PUSH, SW21 SW_PUSH, SW22 SW_PUSH, SW23 SW_PUSH, SW24 SW_PUSH, SW25 SW_PUSH, SW26 SW_PUSH, SW27 SW_PUSH, SW28 SW_PUSH, SW29 SW_PUSH, SW3 SW_PUSH, SW30 SW_PUSH, SW31 SW_PUSH, SW32 SW_PUSH, SW33 SW_PUSH, SW34 SW_PUSH, SW35 SW_PUSH, SW36 SW_PUSH, SW37 SW_PUSH, SW38 SW_PUSH, SW39 SW_PUSH, SW4 SW_PUSH, SW40 SW_PUSH, SW41 SW_PUSH, SW42 SW_PUSH, SW5 SW_PUSH, SW6 SW_PUSH, SW7 SW_PUSH, SW8 SW_PUSH, SW9 SW_PUSH, U1 ProMicro, U2 ProMicro

Commit message: [REL] V1
Parts:
- removed the G*** at (241.0, 91.0)
- removed the G*** at (60.0, 90.9)
- removed the G*** at (240.8, 91.0)
- removed the Ref** at (193.2, 51.9)
- removed the Ref** at (179.5, 99.4)
- removed the Ref** at (226.1, 91.7)
- removed the Ref** at (269.2, 55.4)
- removed the Ref** at (269.2, 74.4)
- removed the Ref** at (50.7, 74.4)
- removed the Ref** at (50.7, 55.4)
- removed the Ref** at (250.2, 74.4)
- removed the Ref** at (250.2, 55.4)
- removed the Ref** at (31.7, 74.4)
- removed the Ref** at (107.7, 51.9)
- removed the Ref** at (31.7, 55.4)
- removed the Ref** at (74.8, 91.7)
- removed the Ref** at (121.4, 99.3)
- added ? (x3): , , F.Cu at (212.0, 86.4)
- added ?: , , F.Cu at (74.5, 110.6)
- added ? (x3): , , F.Cu at (69.5, 48.3)
- added ?: , , F.Cu at (179.2, 118.5)
- added ?: , , F.Cu at (31.5, 55.4)
- added ?: , , F.Cu at (225.7, 110.6)
- added ?: , , F.Cu at (107.4, 51.9)
- added ? (x3): , , F.Cu at (88.4, 86.4)
- added ?: , , F.Cu at (250.0, 74.4)
- added ?: , , F.Cu at (50.5, 74.4)
- added ? (x3): , , F.Cu at (231.0, 48.3)
- added ? (x3): , , F.Cu at (31.5, 93.5)
- added ?: , , B.Cu at (121.0, 118.5)
- added ? (x3): , , F.Cu at (269.0, 93.5)
- added ?: , , F.Cu at (193.0, 51.9)
- added ?: , , F.Cu at (269.0, 55.4)
- added D43: D, kbd:D3_TH, B.Cu at (30.1, 105.1)
- added D44: D, kbd:D3_TH, B.Cu at (32.8, 105.1)
- added D45: D, kbd:D3_TH, B.Cu at (68.0, 98.3)
- added D46: D, kbd:D3_TH, B.Cu at (70.8, 98.3)
- added D47: D, kbd:D3_TH, B.Cu at (106.2, 98.7)
- added D48: D, kbd:D3_TH, B.Cu at (108.9, 98.6)
- added D49: D, kbd:D3_TH, B.Cu at (270.4, 103.7)
- added D50: D, kbd:D3_TH, B.Cu at (267.6, 103.7)
- added D51: D, kbd:D3_TH, B.Cu at (232.3, 98.4)
- added D52: D, kbd:D3_TH, B.Cu at (229.6, 98.4)
- added D53: D, kbd:D3_TH, B.Cu at (194.4, 100.5)
- added D54: D, kbd:D3_TH, B.Cu at (191.5, 100.5)
- added G***: LOGO, kbd:corne-logo-horizontal, B.Cu at (238.0, 110.2)
- added G***: LOGO, kdkb_tools:plus, B.Cu at (54.5, 109.0)
- added G***: LOGO, kdkb_tools:logo-vsmall, B.Cu at (246.5, 110.0)
- added G***: LOGO, kdkb_tools:plus, F.Cu at (245.9, 109.1)
- added G***: LOGO, kbd:corne-logo-horizontal, F.Cu at (239.4, 110.2)
- added G***: LOGO, kdkb_tools:plus, F.Cu at (68.9, 108.9)
- added G***: LOGO, kdkb_tools:logo-vsmall, F.Cu at (230.9, 110.0)
- added G***: LOGO, kdkb_tools:logo-vsmall, F.Cu at (53.9, 109.8)
- added G***: LOGO, kdkb_tools:plus, B.Cu at (231.5, 109.1)
- added G***: LOGO, kdkb_tools:logo-vsmall, B.Cu at (69.5, 109.8)
- added G***: LOGO, kbd:corne-logo-horizontal, B.Cu at (61.0, 110.1)
- added Ref**: Val**, kbd:thread_m2, B.Cu at (50.5, 74.4)
- added Ref**: Val**, kbd:thread_m2, B.Cu at (212.0, 86.4)
- added Ref**: Val**, kbd:thread_m2, B.Cu at (193.0, 51.9)
- added Ref**: Val**, kbd:thread_m2, B.Cu at (31.5, 93.5)
- added Ref**: Val**, kbd:thread_m2, B.Cu at (88.4, 86.4)
- added Ref**: Val**, kbd:thread_m2, B.Cu at (31.5, 55.4)
- added Ref**: Val**, kbd:thread_m2, B.Cu at (231.0, 48.3)
- added Ref**: Val**, kbd:thread_m2, B.Cu at (179.2, 118.5)
- added Ref**: Val**, kbd:thread_m2, B.Cu at (69.5, 48.3)
- added Ref**: Val**, kbd:thread_m2, B.Cu at (269.0, 55.4)
- added Ref**: Val**, kbd:thread_m2, B.Cu at (250.0, 74.4)
- added Ref**: Val**, kbd:thread_m2, F.Cu at (121.0, 118.5)
- added Ref**: Val**, kbd:thread_m2, B.Cu at (225.7, 110.6)
- added Ref**: Val**, kbd:thread_m2, B.Cu at (74.5, 110.6)
- added Ref**: Val**, kbd:thread_m2, B.Cu at (269.0, 93.5)
- added Ref**: Val**, kbd:thread_m2, B.Cu at (107.4, 51.9)
- added SW43: SW_PUSH, kbd:CherryMX_ChocV2_1u, F.Cu at (21.9, 103.0)
- added SW44: SW_PUSH, kbd:CherryMX_ChocV2_1u, F.Cu at (41.0, 103.0)
- added SW45: SW_PUSH, kbd:CherryMX_ChocV2_1u, F.Cu at (59.9, 98.2)
- added SW46: SW_PUSH, kbd:CherryMX_ChocV2_1u, F.Cu at (78.9, 95.9)
- added SW47: SW_PUSH, kbd:CherryMX_ChocV2_1u, F.Cu at (98.0, 98.3)
- added SW48: SW_PUSH, kbd:CherryMX_ChocV2_1u, F.Cu at (117.0, 100.7)
- added SW49: SW_PUSH, kbd:CherryMX_ChocV2_1u, F.Cu at (278.5, 103.0)
- added SW50: SW_PUSH, kbd:CherryMX_ChocV2_1u, F.Cu at (259.5, 103.0)
- added SW51: SW_PUSH, kbd:CherryMX_ChocV2_1u, F.Cu at (240.4, 98.3)
- added SW52: SW_PUSH, kbd:CherryMX_ChocV2_1u, F.Cu at (221.5, 95.9)
- added SW53: SW_PUSH, kbd:CherryMX_ChocV2_1u, F.Cu at (202.5, 98.2)
- added SW54: SW_PUSH, kbd:CherryMX_ChocV2_1u, F.Cu at (183.4, 100.6)
- D1, D10, D11, D12, D13, D14, D15, D16, D17, D18, D19, D2, D20, D21, D22, D23, D24, D25, D26, D27, D28, D29, D3, D30, D31, D32, D33, D34, D35, D36, D37, D38, D39, D4, D40, D41, D42, D5, D6, D7, D8, D9: footprint kbd:D3_TH_SMD_v2 -> kbd:D3_TH
- SW1, SW10, SW11, SW12, SW13, SW14, SW15, SW16, SW17, SW18, SW19, SW2, SW20, SW22, SW23, SW24, SW25, SW26, SW27, SW28, SW29, SW3, SW30, SW31, SW32, SW33, SW34, SW35, SW36, SW37, SW38, SW39, SW4, SW40, SW41, SW5, SW6, SW7, SW8, SW9: footprint kbd:keyswitch_cherrymx_alps_choc12_1u -> kbd:CherryMX_ChocV2_1u
- SW21, SW42: footprint kbd:keyswitch_cherrymx_alps_choc12_1.5u -> kbd:CherryMX_ChocV2_1.5u
- moved G*** 19.2 mm to (62.4, 110.0)
- moved D41 19.1 mm to (203.9, 118.0)
- moved D42 19.1 mm to (200.9, 118.0)
- moved J5 19.1 mm to (21.9, 112.4)
- moved J5 19.1 mm to (59.9, 112.4)
- moved D19 19.1 mm to (80.2, 118.0)
- moved D20 19.1 mm to (96.4, 118.0)
- moved D21 19.1 mm to (99.4, 118.0)
- moved D40 19.1 mm to (219.9, 118.0)
- moved J5 19.1 mm to (278.5, 112.4)
- moved J5 19.1 mm to (240.5, 112.4)
- moved SW19 19.1 mm to (88.4, 117.8)
- moved SW20 19.1 mm to (109.4, 120.6)
- moved SW21 19.1 mm to (131.6, 124.3)
- moved SW40 19.1 mm to (211.9, 117.8)
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Connections:
- J1 pad A: Net-(J1-PadA) -> unconnected-(J1-PadA)
- J6 pad A: Net-(J6-PadA) -> unconnected-(J6-PadA)
- U1 pad 1: Net-(U1-Pad1) -> unconnected-(U1-TX0/D3-Pad1)
- U1 pad 10: row3 -> row4
- U1 pad 11: Net-(U1-Pad11) -> row3
- U1 pad 12: Net-(U1-Pad12) -> unconnected-(U1-9/B5-Pad12)
- U1 pad 13: Net-(U1-Pad13) -> unconnected-(U1-B6/10-Pad13)
- U1 pad 14: Net-(U1-Pad14) -> unconnected-(U1-B2/16-Pad14)
- U1 pad 24: Net-(U1-Pad24) -> unconnected-(U1-RAW-Pad24)
- U2 pad 1: Net-(U2-Pad1) -> unconnected-(U2-TX0/D3-Pad1)
- U2 pad 10: row3_r -> row4_r
- U2 pad 11: Net-(U2-Pad11) -> row3_r
- U2 pad 12: Net-(U2-Pad12) -> unconnected-(U2-9/B5-Pad12)
- U2 pad 13: Net-(U2-Pad13) -> unconnected-(U2-B6/10-Pad13)
- U2 pad 14: Net-(U2-Pad14) -> unconnected-(U2-B2/16-Pad14)
- U2 pad 24: Net-(U2-Pad24) -> unconnected-(U2-RAW-Pad24)
Routing:
- net row4: track 0.00 -> 153.8 mm
- net row4_r: track 0.00 -> 136.0 mm, vias 0 -> 2
- net Net-(D46-A): track 0.00 -> 34.9 mm
- net Net-(D53-A): track 0.00 -> 27.2 mm
- net Net-(D44-A): track 0.00 -> 27.0 mm
- net Net-(D49-A): track 0.00 -> 25.4 mm
- net Net-(D51-A): track 0.00 -> 24.9 mm
- net Net-(D52-A): track 0.00 -> 22.2 mm
- net col1_r: track 161.3 -> 183.0 mm
- net col0: track 182.3 -> 203.9 mm
- net col1: track 156.5 -> 178.0 mm
- net col2_r: track 141.1 -> 162.6 mm
- net col5_r: track 105.6 -> 127.0 mm
- net row3: track 94.6 -> 115.9 mm
- net col0_r: track 183.2 -> 204.5 mm
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Other:
- board size 275.5 x 105.6 mm -> 275.6 x 124.6 mm
- board text removed: "Corne Light v2.0 PCB Designed by foostan"

Commit message: [DEV] Fixes
Routing:
- net Net-(D48-A): track 11.2 -> 23.8 mm
Other:
- rule pad_to_mask_clearance: 0.2 -> 0
Changed lines of the file:
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@@
 	)
 	(setup
-		(pad_to_mask_clearance 0.2)
+		(pad_to_mask_clearance 0)
 		(allow_soldermask_bridges_in_footprints no)
 		(aux_axis_origin 74.8395 91.6855)
@@
 	)
 	(segment
+		(start 120.2625 103.321527)
+		(end 120.2625 96.301527)
+		(width 0.25)
+		(layer "F.Cu")
+		(net 81)
+	)
+	(segment
+		(start 117.0125 106.571527)
+		(end 120.2625 103.321527)
+		(width 0.25)
+		(layer "F.Cu")
+		(net 81)
+	)
+	(segment
+		(start 120.2625 96.301527)
+		(end 119.5525 95.591527)
+		(width 0.25)
+		(layer "F.Cu")
+		(net 81)
+	)
+	(segment
