File: corne-light/pcb/corne-light.kicad_sch (KiCad schematic)
At the start: 92 parts, among them J1 MJ-4PP-9, J2 OLED, J6 MJ-4PP-9, J7 OLED, SW1 SW_PUSH, SW10 SW_PUSH, SW11 SW_PUSH, SW12 SW_PUSH, SW13 SW_PUSH, SW14 SW_PUSH, SW15 SW_PUSH, SW16 SW_PUSH, SW17 SW_PUSH, SW18 SW_PUSH, SW19 SW_PUSH, SW2 SW_PUSH, SW20 SW_PUSH, SW21 SW_PUSH, SW22 SW_PUSH, SW23 SW_PUSH, SW24 SW_PUSH, SW25 SW_PUSH, SW26 SW_PUSH, SW27 SW_PUSH, SW28 SW_PUSH, SW29 SW_PUSH, SW3 SW_PUSH, SW30 SW_PUSH, SW31 SW_PUSH, SW32 SW_PUSH, SW33 SW_PUSH, SW34 SW_PUSH, SW35 SW_PUSH, SW36 SW_PUSH, SW37 SW_PUSH, SW38 SW_PUSH, SW39 SW_PUSH, SW4 SW_PUSH, SW40 SW_PUSH, SW41 SW_PUSH, SW42 SW_PUSH, SW5 SW_PUSH, SW6 SW_PUSH, SW7 SW_PUSH, SW8 SW_PUSH, SW9 SW_PUSH, U1 ProMicro, U2 ProMicro

Commit message: [REL] KA v1
Parts:
- added D43, D44, D45, D46, D47, D48: D, kbd:D3_TH, symbol Device:D
- added SW43, SW44, SW45, SW46, SW47, SW48: SW_PUSH, kbd:CherryMX_ChocV2_1u, symbol kbd:SW_PUSH
Connections:
- net col0: now also SW43.1; no longer SW13.1
- net col3: now also SW46.1
- net col4: now also SW47.1
- net col5: now also SW48.1
- net row3: now also D43.1 (K), D44.1 (K), D45.1 (K), D46.1 (K), D47.1 (K), D48.1 (K); no longer D19.1 (K), D20.1 (K), D21.1 (K)
- net row3_r: no longer D40.1 (K), D41.1 (K), D42.1 (K)
- new net: D47.2 (A), SW47.2
- new net: D46.2 (A), SW46.2
- new net: D45.2 (A), SW45.2
- new net: D43.2 (A), SW43.2
- new net: D44.2 (A), SW44.2
- new net: D48.2 (A), SW48.2
- new net row4: D19.1 (K), D20.1 (K), D21.1 (K)
- new net row4_r: D40.1 (K), D41.1 (K), D42.1 (K)
- no-connect marks 15 -> 13
Other:
- moved on the sheet: D19, D20, D21, SW19, SW20, SW21
