File: corne-light/pcb/corne-light.kicad_sch (KiCad schematic)
At the start: 92 parts, among them J1 MJ-4PP-9, J2 OLED, J6 MJ-4PP-9, J7 OLED, SW1 SW_PUSH, SW10 SW_PUSH, SW11 SW_PUSH, SW12 SW_PUSH, SW13 SW_PUSH, SW14 SW_PUSH, SW15 SW_PUSH, SW16 SW_PUSH, SW17 SW_PUSH, SW18 SW_PUSH, SW19 SW_PUSH, SW2 SW_PUSH, SW20 SW_PUSH, SW21 SW_PUSH, SW22 SW_PUSH, SW23 SW_PUSH, SW24 SW_PUSH, SW25 SW_PUSH, SW26 SW_PUSH, SW27 SW_PUSH, SW28 SW_PUSH, SW29 SW_PUSH, SW3 SW_PUSH, SW30 SW_PUSH, SW31 SW_PUSH, SW32 SW_PUSH, SW33 SW_PUSH, SW34 SW_PUSH, SW35 SW_PUSH, SW36 SW_PUSH, SW37 SW_PUSH, SW38 SW_PUSH, SW39 SW_PUSH, SW4 SW_PUSH, SW40 SW_PUSH, SW41 SW_PUSH, SW42 SW_PUSH, SW5 SW_PUSH, SW6 SW_PUSH, SW7 SW_PUSH, SW8 SW_PUSH, SW9 SW_PUSH, U1 ProMicro, U2 ProMicro

Commit message: [REL] V1
Parts:
- added D43, D44, D45, D46, D47, D48, D49, D50, D51, D52, D53, D54: D, kbd:D3_TH, symbol Device:D
- added SW43, SW44, SW45, SW46, SW47, SW48, SW49, SW50, SW51, SW52, SW53, SW54: SW_PUSH, kbd:CherryMX_ChocV2_1u, symbol kbd:SW_PUSH
Connections:
- net col0: now also SW43.1
- net col0_r: now also SW49.1
- net col1: now also SW44.1
- net col1_r: now also SW50.1
- net col2: now also SW45.1
- net col2_r: now also SW51.1
- net col3: now also SW46.1
- net col3_r: now also SW52.1
- net col4: now also SW47.1
- net col4_r: now also SW53.1
- net col5: now also SW48.1
- net col5_r: now also SW54.1
- net row3: now also U1.11 (8/B4); no longer U1.10 (7/E6)
- net row3_r: now also U2.11 (8/B4); no longer U2.10 (7/E6)
- new net: D52.2 (A), SW52.2
- new net: D43.2 (A), SW43.2
- new net: D49.2 (A), SW49.2
- new net: D54.2 (A), SW54.2
- new net: D53.2 (A), SW53.2
- new net: D44.2 (A), SW44.2
- new net: D45.2 (A), SW45.2
- new net: D48.2 (A), SW48.2
- new net: D51.2 (A), SW51.2
- new net: D46.2 (A), SW46.2
- new net: D50.2 (A), SW50.2
- new net: D47.2 (A), SW47.2
- new net row4: D43.1 (K), D44.1 (K), D45.1 (K), D46.1 (K), D47.1 (K), D48.1 (K), U1.10 (7/E6)
- new net row4_r: D49.1 (K), D50.1 (K), D51.1 (K), D52.1 (K), D53.1 (K), D54.1 (K), U2.10 (7/E6)
- no-connect marks 15 -> 14
Other:
- company: foostan -> KDKB - foostan
- title: Corne Light -> Corne Light+
- moved on the sheet: D1, D10, D11, D12, D13, D14, D15, D16, D17, D18, D19, D2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
